File: XiaoSeeedBLE001.kicad_sch (KiCad schematic)
At the start: 1 part

Commit message: jdkjfskdfk
kgkejk
Parts:
- added SW? (x17): SW_Push, symbol Switch:SW_Push
- added SW? (x3): (no value), symbol Switch:SW_Push
- U?: value (none) -> SeeeduinoXIAO

Commit message: kmmkk
Parts:
- removed SW? (x16): SW_Push, symbol Switch:SW_Push
- added D1, D10, D11, D12, D13, D14, D15, D16, D17, D18, D19, D2, D20, D21, D22, D23, D24, D25, D26, D3, D4, D5, D6, D7, D8, D9: 1N4448W, Diode_SMD:D_SOD-123, symbol Diode:1N4448W
- added SW10, SW11, SW12, SW13, SW14, SW15, SW16, SW17, SW18, SW19, SW20, SW21, SW22, SW23, SW24, SW25, SW26, SW7, SW8, SW9: SW_Push, BOB_Pretty_Master_MOFO_UWU:Kailh_socket_PG1350_optional, symbol Switch:SW_Push
- added SW27: SW_SPDT, Button_Switch_SMD:SW_SPDT_PCM12, symbol Switch:SW_SPDT
- added SW5, SW6: SW_Push, symbol Switch:SW_Push
- SW1, SW2, SW3: renamed from SW?; value (none) -> SW_Push
- U1: renamed from U?; footprint (none) -> Seeeduino XIAO KICAD:Seeeduino XIAO-MOUDLE14P-2.54-21X17.8MM
- gave numbers to parts that had none: 1
Connections:
- net col3: now reaches SW3.1
- net col3: now also SW10.1, SW17.1, SW24.1
- net at SW3.2: now also D3.2 (A)
- net col2: now reaches SW2.1
- net col2: now also SW16.1, SW23.1, SW9.1
- net at SW2.2: now also D2.2 (A)
- net col1: now reaches SW1.1
- net col1: now also SW15.1, SW22.1, SW8.1
- net at SW1.2: now also D1.2 (A)
- net col4: now reaches SW4.1
- net col4: now also SW11.1, SW18.1, SW25.1
- net at SW4.2: now also D4.2 (A)
- new net: D8.2 (A), SW8.2
- new net: D23.2 (A), SW23.2
- new net: D13.2 (A), SW13.2
- new net: D24.2 (A), SW24.2
- new net: D12.2 (A), SW12.2
- new net: D18.2 (A), SW18.2
- new net: D9.2 (A), SW9.2
- new net: D16.2 (A), SW16.2
- new net: D22.2 (A), SW22.2
- new net: D19.2 (A), SW19.2
- new net: D7.2 (A), SW7.2
- new net: D5.2 (A), SW5.2
- new net: D21.2 (A), SW21.2
- new net: D20.2 (A), SW20.2
- new net: D15.2 (A), SW15.2
- new net: D11.2 (A), SW11.2
- new net: D10.2 (A), SW10.2
- new net: D25.2 (A), SW25.2
- new net: D17.2 (A), SW17.2
- new net: D6.2 (A), SW6.2
- new net: D14.2 (A), SW14.2
- new net: D26.2 (A), SW26.2
- new net col5: SW12.1, SW19.1, SW26.1, SW5.1
- new net col6: SW13.1, SW20.1, SW6.1
- new net col7: SW14.1, SW21.1, SW7.1
- new net row1: D1.1 (K), D2.1 (K), D3.1 (K), D4.1 (K), D5.1 (K), D6.1 (K), D7.1 (K)
- new net row2: D10.1 (K), D11.1 (K), D12.1 (K), D13.1 (K), D14.1 (K), D8.1 (K), D9.1 (K)
- new net row3: D15.1 (K), D16.1 (K), D17.1 (K), D18.1 (K), D19.1 (K), D20.1 (K), D21.1 (K)
- new net row4: D22.1 (K), D23.1 (K), D24.1 (K), D25.1 (K), D26.1 (K)
Other:
- moved on the sheet: SW1, SW2, SW3, SW4, U1
